File: WaterLevelDetector_v5_tiny_icsp.kicad_pcb (KiCad board)
At the start: 2 copper layers, 31.8 x 58.8 mm, 12 parts, among them J3 USB_C_Receptacle_PowerOnly_6P, J4 Conn_02x03_Odd_Even, U1 ATtiny85-20P

Commit message: updated pcb to have gnd gpio vcc
Other:
- board text added: "VCC GPIO GND"
